Commit message: Aggiunti i tag di gazebo per la simulazione

File: description/robot.urdf.xacro (robot description, xacro)
@@ -4,3 +4,6 @@
     <!-- Con questa riga di codice stiamo richiamando il file che contiene la struttura di base -->
     <xacro:include filename="robot_core.xacro" />
+    <!-- Con questa riga andremo ad includere il file che contiene le righe di codice per utilizzare il controllo
+         di Gazebo -->
+    <xacro:include filename="gazebo_control.xacro"/>
 </robot>

File: description/robot_core.xacro (robot description, xacro)
@@ -62,4 +62,8 @@
             </xacro:inertial_box>
         </link>
+        <!-- Andiamo ad aggiungere le TAG per GAZEBO affinchè riesca a funzionare senza problemi, specifichiamo il colore-->
+        <gazebo reference="chassis">
+            <material>Gazebo/White</material>
+        </gazebo>
         <!-- adesso iniziamo definendo le ruote del nostro robot, che connetteremo alla terna base,
              perche quella risulta essere il centro di rotazione del nostro robot e bisognerà
@@ -91,4 +95,7 @@
             </xacro:inertial_cylinder>
         </link>
+        <gazebo reference="left_wheel">
+            <material>Gazebo/Blue</material>
+        </gazebo>
         <!-- RUOTA DESTRA -->
         <joint name="right_wheel_joint" type="continuous">
@@ -114,4 +121,7 @@
             </xacro:inertial_cylinder>
         </link>
+        <gazebo reference="right_wheel">
+            <material>Gazebo/Blue</material>
+        </gazebo>
         <!-- Adesso vogliamo realizzare la ruotina folle, prenderemo alcuni accorgimenti, cioè quello di considerarla senza attrito per semplicità,
              non è del tutto corretto, ma stiamo semplificando il problema-->
@@ -138,3 +148,9 @@
             </xacro:inertial_sphere>
         </link>
+        <gazebo reference="caster_wheel">
+            <material>Gazebo/Black</material>
+            <!-- possiamo impostare anche i coefficenti di attrito per i link -->
+            <mu1 value="0.001"/>
+            <mu2 value="0.001"/>
+        </gazebo>
 </robot>

Commit message: Aggiunto il sensore Lidar

File: description/robot.urdf.xacro (robot description, xacro)
@@ -7,3 +7,5 @@
          di Gazebo -->
     <xacro:include filename="gazebo_control.xacro"/>
+    <!-- Inseriamo il file che si occuperà di far funzionare il sensore LIDAR sul nostro robot simulato -->
+    <xacro:include filename="lidar.xacro"/>
 </robot>

File: description/robot_core.xacro (robot description, xacro)
@@ -18,4 +18,7 @@
     <material name="black">
         <color rgba="0 0 0 1" />
+    </material>
+    <material name="red">
+        <color rgba="1 0 0 1" />
     </material>
     <!-- Adesso iniziamo la sezione dove decriviamo i link che avrà il nostro robot,

Commit message: Vari FIX

File: description/robot.urdf.xacro (robot description, xacro)
@@ -2,12 +2,19 @@
 <robot xmlns:xacro="http://www.ros.org/wiki/xacro"  name="robot">
     <!-- In questo file andremo a richiamare tutti gli altri file URDF che contengono le varie parti del robot-->
-    <!-- Con questa riga di codice stiamo richiamando il file che contiene la struttura di base -->
+     <!-- Con questa riga di codice stiamo richiamando il file che contiene la struttura di base -->
     <xacro:include filename="robot_core.xacro" />
-    <!-- Con questa riga andremo ad includere il file che contiene le righe di codice per utilizzare il controllo
-         di Gazebo -->
-    <!-- <xacro:include filename="gazebo_control.xacro"/> -->
+    <!--                                         SCELTA CONTROLLO                                    -->
+    <xacro:arg name="use_ros2_control" default="true"/>
+    <xacro:if value="$(arg use_ros2_control)">
     <!-- Con questa riga andremo ad includere il file che contiene le righe di codice per utilizzare il controllo
          di ROS2_CONTROL -->
      <xacro:include filename="ros2_control.xacro"/>
+    </xacro:if>
+    <xacro:unless value="$(arg use_ros2_control)">
+    <!-- Con questa riga andremo ad includere il file che contiene le righe di codice per utilizzare il controllo
+     di Gazebo -->
+    <xacro:include filename="gazebo_control.xacro"/>
+    </xacro:unless>
+    <!--                                           SENSORI                                                    -->
     <!-- Inseriamo il file che si occuperà di far funzionare il sensore LIDAR sul nostro robot simulato -->
     <xacro:include filename="lidar.xacro"/>

File: description/robot_core.xacro (robot description, xacro)
@@ -91,5 +91,5 @@
             <collision>
                 <geometry>
-                    <cylinder radius="0.05" length="0.04"/>
+                    <sphere radius="0.05"/>
                 </geometry>
             </collision>
@@ -117,5 +117,5 @@
             <collision>
                 <geometry>
-                    <cylinder radius="0.05" length="0.04"/>
+                    <sphere radius="0.05"/>
                 </geometry>
             </collision>
