Commit message: Aggiungo SLAM_toolbox

File: description/robot_core.xacro (robot description, xacro)
@@ -30,4 +30,14 @@
          <link name="base_link">
          </link>
+         <!-- Dobbiamo aggiungere quel link fittizio che serve per utilizzare l'algoritmo di SLAM, che
+              sarà coincidente con il base link -->
+        <!-- BASE_FOOTPRINT LINK -->
+        <joint name="base_footprint_joint" type="fixed">
+            <parent link="base_link"/>
+            <child link="base_footprint"/>
+            <origin xyz="0 0 0" rpy="0 0 0"/>
+        </joint>
+        <link name="base_footprint">
+        </link>
          <!-- Come prossimo obbiettivo dobbiamo stabilire le dimensioni del nostro robot,
               supporremo LARGHEZZA= 300 mm , LUNGHEZZA= 300 mm , ALTEZZA = 150 mm .
